File: solar-car.kicad_pcb (KiCad board)
At the start: 2 copper layers, 78.7 x 91.4 mm, 22 parts, among them J1 Motor Out, J2 Solar In, Q1 BS270, Q2 BS250, Q3 IPP034N03L, U1 TL494

Commit message: filled in rows
Connections:
- U1 pad 8: unconnected-(U1-C1-Pad8) -> Net-(U1-C1)
- U1 pad 9: unconnected-(U1-E1-Pad9) -> Net-(U1-C1)
Routing:
- net (no net): track 0.00 -> 368.3 mm
- net GND: track 269.3 -> 353.1 mm
- net Net-(U1-C1): track 0.00 -> 73.7 mm
- net Net-(J1-Pin_1): track 35.6 -> 27.9 mm
- net +5V: track 76.2 -> 71.1 mm
- net VCC: track 261.6 -> 259.1 mm
Changed lines of the file:
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@@
 			(layers "*.Cu" "*.Mask")
 			(remove_unused_layers no)
-			(net "unconnected-(U1-C1-Pad8)")
+			(net "Net-(U1-C1)")
 			(pinfunction "C1_8")
-			(pintype "passive+no_connect")
+			(pintype "passive")
 		)
 		(pad "9" thru_hole circle
@@
 			(layers "*.Cu" "*.Mask")
 			(remove_unused_layers no)
-			(net "unconnected-(U1-E1-Pad9)")
+			(net "Net-(U1-C1)")
 			(pinfunction "E1_9")
-			(pintype "passive+no_connect")
+			(pintype "passive")
 		)
 		(pad "10" thru_hole circle
@@
 		(sheetname "/")
 		(sheetfile "solar-car.kicad_sch")
+		(units
+			(unit
+				(name "A")
+				(pins "1" "2")
+			)
+		)
 		(attr through_hole)
 		(duplicate_pad_numbers_are_jumpers no)
@@
 	)
 	(segment
+		(start 93.98 109.22)
+		(end 167.64 109.22)
+		(width 2)
+		(layer "B.Cu")
+		(net "")
+	)
+	(segment
+		(start 93.98 111.76)
+		(end 167.64 111.76)
+		(width 2)
+		(layer "B.Cu")
+		(net "")
+	)
+	(segment
+		(start 167.64 55.88)
+		(end 93.98 55.88)
+		(width 2)
+		(layer "B.Cu")
+		(net "")
+	)
+	(segment
+		(start 93.98 99.06)
+		(end 167.64 99.06)
+		(width 2)
+		(layer "B.Cu")
+		(net "")
+	)
+	(segment
+		(start 167.64 96.52)
+		(end 93.98 96.52)
+		(width 2)
+		(layer "B.Cu")
+		(net "")
+	)
+	(segment
 		(start 167.64 73.66)
 		(end 167.64 50.8)
@@
 	)
 	(segment
-		(start 157.48 88.9)
-		(end 154.94 88.9)
-		(width 2)
-		(layer "B.Cu")
-		(net "VCC")
-	)
-	(segment
 		(start 109.22 114.3)
 		(end 139.7 114.3)
@@
 	)
 	(segment
+		(start 93.98 53.34)
+		(end 167.64 53.34)
+		(width 2)
+		(layer "B.Cu")
+		(net "GND")
+	)
+	(segment
 		(start 134.62 83.82)
 		(end 93.98 83.82)
@@
 	)
 	(segment
+		(start 144.78 83.82)
+		(end 167.64 83.82)
+		(width 2)
+		(layer "B.Cu")
+		(net "GND")
+	)
+	(segment
 		(start 139.7 88.9)
 		(end 142.24 88.9)
@@
 	)
 	(segment
-		(start 147.32 88.9)
-		(end 149.86 88.9)
-		(width 2)
-		(layer "B.Cu")
-		(net "GND")
-	)
-	(segment
 		(start 147.24 83.82)
 		(end 147.32 83.74)
@@
 	)
 	(segment
-		(start 116.84 106.68)
-		(end 127 106.68)
-		(width 2)
-		(layer "B.Cu")
-		(net "GND")
-	)
-	(segment
 		(start 152.4 101.6)
 		(end 167.64 101.6)
@@
 	)
 	(segment
-		(start 139.7 106.68)
-		(end 132.08 106.68)
-		(width 2)
-		(layer "B.Cu")
-		(net "Net-(J1-Pin_1)")
-	)
-	(segment
 		(start 165.1 106.68)
 		(end 139.7 106.68)
@@
 	)
 	(segment
-		(start 149.86 66.04)
-		(end 132.08 66.04)
+		(start 147.32 73.66)
+		(end 147.32 66.04)
 		(width 2)
 		(layer "F.Cu")
@@
 	)
 	(segment
-		(start 132.08 66.04)
-		(end 132.08 68.58)
+		(start 147.32 66.04)
+		(end 132.08 66.04)
 		(width 2)
 		(layer "F.Cu")
@@
 	)
 	(segment
-		(start 149.86 73.66)
-		(end 149.86 66.04)
+		(start 132.08 66.04)
+		(end 132.08 68.58)
 		(width 2)
 		(layer "F.Cu")
@@
 	)
 	(via
-		(at 149.86 73.66)
+		(at 147.32 73.66)
 		(size 0.6)
 		(drill 1)
@@
 	)
 	(segment
-		(start 142.24 73.66)
-		(end 147.32 73.66)
+		(start 147.32 73.66)
+		(end 142.24 73.66)
 		(width 2)
 		(layer "B.Cu")
@@
 	)
 	(segment
-		(start 147.32 73.66)
-		(end 149.86 73.66)
+		(start 142.24 86.36)
+		(end 167.64 86.36)
 		(width 2)
 		(layer "B.Cu")
-		(net "+5V")
+		(net "Net-(U1-C1)")
+	)
+	(segment
+		(start 134.62 86.36)
+		(end 93.98 86.36)
+		(width 2)
+		(layer "B.Cu")
+		(net "Net-(U1-C1)")
+	)
+	(segment
+		(start 134.62 86.36)
+		(end 142.24 86.36)
+		(width 2)
+		(layer "B.Cu")
+		(net "Net-(U1-C1)")
 	)
 	(embedded_fonts no)

Commit message: irl changes
Parts:
- added C6: 220u, Capacitor_THT:CP_Radial_D6.3mm_P2.50mm, F.Cu at (142.2, 50.8)
- added C7: 100n, Capacitor_THT:CP_Radial_D6.3mm_P2.50mm, F.Cu at (127.0, 50.8)
- C1: value C_Small -> 100n
- R8: value R -> 10k
- R9: value R_Small -> 100k
