File: solar-car.kicad_sch (KiCad schematic)
At the start: 22 parts, among them J1 Motor Out, J2 Solar In, Q1 BS270, Q2 BS250, Q3 IPP034N03L, U1 TL494

Commit message: filled in rows
Connections:
- net at U1.8 (C1): now also U1.9 (E1)
- no-connect marks 2 -> 0
Changed lines of the file:
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@@
 		(color 0 0 0 0)
 	)
-	(no_connect
-		(at 120.65 77.47)
-	)
-	(no_connect
-		(at 120.65 85.09)
-	)
 	(wire
 		(pts
@@
 	(wire
 		(pts
+			(xy 121.92 77.47) (xy 121.92 85.09)
+		)
+		(stroke
+			(width 0)
+			(type default)
+		)
+	)
+	(wire
+		(pts
 			(xy 95.25 85.09) (xy 77.47 85.09)
 		)
@@
 	(wire
 		(pts
+			(xy 120.65 77.47) (xy 121.92 77.47)
+		)
+		(stroke
+			(width 0)
+			(type default)
+		)
+	)
+	(wire
+		(pts
 			(xy 124.46 80.01) (xy 134.62 80.01)
 		)
@@
 		)
 		(stroke
+			(width 0)
+			(type default)
+		)
+	)
+	(wire
+		(pts
+			(xy 121.92 85.09) (xy 120.65 85.09)
+		)
+		(stroke

Commit message: irl changes
Parts:
- added C6: 220u, Capacitor_THT:CP_Radial_D6.3mm_P2.50mm, symbol Device:C_Polarized
- added C7: 100n, Capacitor_THT:CP_Radial_D6.3mm_P2.50mm, symbol Device:C
- C1: value C_Small -> 100n
- R8: value R -> 10k
- R9: value R_Small -> 100k
Connections:
- net GND: now also C6.2, C7.2
- net VCC: now also C6.1, C7.1
Other:
- moved on the sheet: C1, C2, C3, C4, C5, D1, J1, J2, L1, Q1, Q2, Q3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
